File: xmas22_hw.kicad_pcb (KiCad board)
At the start: 2 copper layers, 60 x 69.5 mm, 46 parts, among them IC1 PIC16F18044-I_ML, J1 Aux side, J2 Main Side, SW1 SW_MEC_5E

Commit message: wip
Parts:
- R9: moved to B.Cu
- SW1: value SW_MEC_5E -> SW_Push; footprint Button_Switch_SMD:SW_Push_1P1T_NO_6x6mm_H9.5mm -> Button_Switch_SMD:SW_SPST_TL3342; moved to B.Cu
- moved C1 80.9 mm to (73.1, 75.3)
- moved D11 80.9 mm to (82.9, 79.6)
- moved D12 80.9 mm to (82.9, 124.1)
- moved D13 80.9 mm to (40.6, 110.4), turned to 108 degrees
- moved D14 80.9 mm to (92.9, 93.4)
- moved D15 80.9 mm to (92.9, 110.4)
- moved D16 80.9 mm to (40.6, 93.4), turned to 72 degrees
- moved IC1 80.9 mm to (75.9, 78.0)
- moved J2 80.9 mm to (66.7, 80.4)
- moved NT1 80.9 mm to (69.4, 73.3)
- moved NT2 80.9 mm to (71.1, 73.3)
- moved R10 80.9 mm to (46.9, 82.8)
- moved R11 80.9 mm to (54.7, 126.6)
- moved R13 80.9 mm to (86.5, 121.0)
- moved R14 80.9 mm to (42.4, 114.8)
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Connections:
- D10 pad 1: GND -> Net-(D10-Pad1)
- D10 pad 2: Net-(D10-Pad2) -> /Main Half/LED_1
- D13 pad 1: GND -> Net-(D13-Pad1)
- D13 pad 2: Net-(D13-Pad2) -> /Main Half/LED_4
- D16 pad 1: GND -> Net-(D16-Pad1)
- D16 pad 2: Net-(D16-Pad2) -> /Main Half/LED_7
- D9 pad 1: GND -> Net-(D9-Pad1)
- D9 pad 2: Net-(D9-Pad2) -> /Main Half/LED_0
- IC1 pad 10: /Main Half/LED_2 -> /Main Half/LED_5
- IC1 pad 11: /Main Half/USER_BTN -> /Main Half/LED_3
- IC1 pad 12: /Main Half/LED_7 -> /Main Half/LED_6
- IC1 pad 13: /Main Half/LED_6 -> /Main Half/LED_2
- IC1 pad 14: /Main Half/LED_5 -> /Main Half/LED_7
- IC1 pad 15: /Main Half/LED_1 -> /Main Half/LED_4
- IC1 pad 19: /Main Half/LED_4 -> /Main Half/LED_1
- IC1 pad 20: /Main Half/LED_3 -> /Main Half/USER_BTN
- NT2 pad 2: /Main Half/LED_1 -> /Main Half/LED_4
- R10 pad 1: Net-(D9-Pad2) -> Net-(D9-Pad1)
- R10 pad 2: /Main Half/LED_0 -> GND
- R11 pad 1: Net-(D10-Pad2) -> Net-(D10-Pad1)
- R11 pad 2: /Main Half/LED_1 -> GND
- R14 pad 1: Net-(D13-Pad2) -> Net-(D13-Pad1)
- R14 pad 2: /Main Half/LED_4 -> GND
- R17 pad 1: Net-(D16-Pad2) -> Net-(D16-Pad1)
- R17 pad 2: /Main Half/LED_7 -> GND
- SW1 pad 2: GND -> /Main Half/USER_BTN
- TP3 pad 1: /Main Half/VSS -> GND
Routing:
- net +3V0: track 2.30 -> 79.9 mm, vias 0 -> 3
- net /Main Half/LED_1: track 0.00 -> 73.6 mm, vias 0 -> 1
- net /Main Half/LED_4: track 0.00 -> 62.8 mm, vias 0 -> 2
- net /Main Half/USER_BTN: track 0.00 -> 55.5 mm, vias 0 -> 1
- net /Main Half/LED_3: track 0.00 -> 54.7 mm
- net /Main Half/LED_7: track 0.00 -> 46.0 mm, vias 0 -> 1
- net (no net): track 45.9 -> 0.00 mm
- net /Main Half/LED_6: track 0.00 -> 37.3 mm, vias 0 -> 1
- net /Main Half/LED_0: track 0.00 -> 27.6 mm, vias 0 -> 2
- net /Main Half/LED_5: track 0.00 -> 16.8 mm
- net GND: track 0.00 -> 13.5 mm, vias 0 -> 22
- net Net-(D13-Pad1): track 0.00 -> 3.01 mm
- net Net-(D14-Pad2): track 0.00 -> 3.01 mm
- net Net-(D16-Pad1): track 0.00 -> 3.01 mm
- net Net-(D9-Pad1): track 0.00 -> 3.01 mm
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- added copper zone on B.Cu, net GND
- added copper zone on F.Cu, net GND

Commit message: wip
Parts:
- D5, D6, D7, D8, R5, R6, R7, R8: moved to B.Cu
- SW1: footprint Button_Switch_SMD:SW_SPST_TL3342 -> Button_Switch_SMD:SW_SPST_B3U-3000P
- moved D4 128.3 mm to (129.5, 110.6), turned to -72 degrees
- moved R4 125.2 mm to (131.4, 115.0), turned to -62 degrees
- moved D8 117.7 mm to (139.5, 124.3), turned to -36 degrees
- moved D7 117.5 mm to (129.5, 93.6), turned to 72 degrees
- moved R7 115.9 mm to (128.5, 98.3), turned to -98 degrees
- moved J1 113.5 mm to (158.0, 80.4)
- moved D2 112.8 mm to (171.9, 124.3), turned to 36 degrees
- moved R8 111.8 mm to (143.6, 126.8), turned to -26 degrees
- moved R3 106.4 mm to (135.9, 83.0), turned to -134 degrees
- moved D3 106.3 mm to (139.5, 79.9), turned to 36 degrees
- moved R2 105.4 mm to (175.5, 121.2), turned to 46 degrees
- moved D6 78.7 mm to (181.9, 110.6), turned to 72 degrees
- moved R6 71.3 mm to (182.9, 105.9), turned to 82 degrees
- moved D5 71.1 mm to (171.9, 79.9), turned to 144 degrees
- moved R5 69.2 mm to (167.8, 77.4), turned to 154 degrees
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Connections:
- D3 pad 1: GND -> Net-(D3-Pad1)
- D3 pad 2: Net-(D3-Pad2) -> /Main Half/AUX_LED_10
- D7 pad 1: GND -> Net-(R7-Pad1)
- D7 pad 2: Net-(D7-Pad2) -> /Main Half/AUX_LED_14
- J1 pad 5: /Main Half/AUX_LED_10 -> /Main Half/AUX_LED_11
- J1 pad 6: /Main Half/AUX_LED_14 -> /Main Half/AUX_LED_15
- J1 pad 7: /Main Half/AUX_LED_11 -> /Main Half/AUX_LED_10
- J1 pad 8: /Main Half/AUX_LED_15 -> /Main Half/AUX_LED_14
- R1 pad 1: /Main Half/AUX_LED_8 -> Net-(D1-Pad2)
- R1 pad 2: Net-(D1-Pad2) -> /Main Half/AUX_LED_8
- R2 pad 1: /Main Half/AUX_LED_9 -> Net-(D2-Pad2)
- R2 pad 2: Net-(D2-Pad2) -> /Main Half/AUX_LED_9
- R3 pad 1: /Main Half/AUX_LED_10 -> Net-(D3-Pad1)
- R3 pad 2: Net-(D3-Pad2) -> GND
- R4 pad 1: /Main Half/AUX_LED_11 -> Net-(D4-Pad2)
- R4 pad 2: Net-(D4-Pad2) -> /Main Half/AUX_LED_11
- R5 pad 1: /Main Half/AUX_LED_12 -> Net-(D5-Pad2)
- R5 pad 2: Net-(D5-Pad2) -> /Main Half/AUX_LED_12
- R6 pad 1: /Main Half/AUX_LED_13 -> Net-(D6-Pad2)
- R6 pad 2: Net-(D6-Pad2) -> /Main Half/AUX_LED_13
- R7 pad 1: /Main Half/AUX_LED_14 -> Net-(R7-Pad1)
- R7 pad 2: Net-(D7-Pad2) -> GND
- R8 pad 1: /Main Half/AUX_LED_15 -> Net-(D8-Pad2)
- R8 pad 2: Net-(D8-Pad2) -> /Main Half/AUX_LED_15
Routing:
- net /Main Half/AUX_LED_14: track 0.00 -> 84.3 mm
- net /Main Half/AUX_LED_11: track 0.00 -> 76.1 mm
- net /Main Half/AUX_LED_9: track 0.00 -> 67.0 mm
- net /Main Half/AUX_LED_10: track 0.00 -> 61.4 mm
- net /Main Half/AUX_LED_15: track 0.00 -> 58.2 mm
- net /Main Half/AUX_LED_13: track 0.00 -> 50.8 mm
- net /Main Half/AUX_LED_8: track 0.00 -> 34.5 mm
- net /Main Half/AUX_LED_12: track 0.00 -> 17.3 mm
- net Net-(D1-Pad2): track 0.00 -> 3.01 mm
- net Net-(D4-Pad2): track 0.00 -> 3.01 mm
- net Net-(D6-Pad2): track 0.00 -> 3.01 mm
- net Net-(R7-Pad1): track 0.00 -> 3.01 mm
- net Net-(D2-Pad2): track 0.00 -> 3.01 mm
- net Net-(D3-Pad1): track 0.00 -> 3.01 mm
- net Net-(D8-Pad2): track 0.00 -> 3.01 mm
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Other:
- board size 60 x 69.5 mm -> 149 x 69.7 mm

Commit message: final run
Parts:
- removed D13: LED, LED_SMD:LED_0603_1608Metric_Pad1.05x0.95mm_HandSolder
- removed R14: R_Small, Resistor_SMD:R_0603_1608Metric_Pad0.98x0.95mm_HandSolder
- BT1: value CR1620 -> CR2032; footprint xmas22:BH57A-5 -> BAT-HLD-001:BATHLD001
- SW1: footprint Button_Switch_SMD:SW_SPST_B3U-3000P -> Button_Switch_SMD:SW_SPST_EVQP0
- moved BT1 1.13 mm to (52.8, 112.5), turned to 180 degrees
Connections:
- net /Main Half/LED_4 renamed Net-(IC1-Pad15)
Routing:
- net Net-(IC1-Pad15): track 62.8 -> 6.76 mm
- net +3V0: track 79.9 -> 57.3 mm
- net /Main Half/!MCLR: track 0.00 -> 17.1 mm, vias 0 -> 1
- net Net-(D13-Pad1): track 3.01 -> 0.00 mm
- net Net-(D15-Pad2): track 0.00 -> 3.01 mm
- net Net-(D11-Pad2): track 0.00 -> 3.01 mm
- net GND: track 13.5 -> 10.5 mm, vias 28 -> 36
- net /Main Half/LED_7: track 46.0 -> 46.8 mm, vias 1 -> 3
- net /Main Half/LED_1: track 73.6 -> 74.2 mm
